Commit message: joy gear shifting added, intersection rebuild with road but the texture is not working in rviz

File: src/prius_description/urdf/prius.urdf (robot description, URDF)
Before this commit: robot solab_prius, 24 links, 23 joints
Joints:
- joint back_camera_joint: origin xyz=0 1.45 1.4 rpy=0 0.05 1.5707 -> xyz=0 1.45 1.4 rpy=0 0.1 1.5707
- joint front_camera_joint: origin xyz=0 -0.4 1.4 rpy=0 0.05 -1.5707 -> xyz=0.17 -0.3 1.3 rpy=0 0.05 -1.5707
- joint left_camera_joint: origin xyz=1 -0.7 1.0 rpy=0 0.05 1.0 -> xyz=0.17 -0.3 1.3 rpy=0 0.05 -0.14
- joint right_camera_joint: origin xyz=-1 -0.7 1.0 rpy=0 0.05 2.1416 -> xyz=0.17 -0.3 1.3 rpy=0 0.05 -3.0

Commit message: testing multi robot

File: src/prius_description/urdf/prius.urdf (robot description, URDF)
Before this commit: robot solab_prius, 24 links, 23 joints
Joints:
- joint front_left_laser_joint: origin xyz=1 -2.3 0.5 rpy=0 0.05 0 -> xyz=1 -2.3 0.5 rpy=0 0.0 0

Commit message: with rosbag

File: src/prius_description/urdf/prius.urdf (robot description, URDF)
Before this commit: robot solab_prius, 24 links, 23 joints
Joints:
- joint front_camera_joint: origin xyz=0.17 -0.3 1.3 rpy=0 0.05 -1.5707 -> xyz=0.17 -0.2 1.3 rpy=0 0.05 -1.5707
- joint left_camera_joint: origin xyz=0.17 -0.3 1.3 rpy=0 0.05 -0.14 -> xyz=0.22 -0.2 1.15 rpy=0 0.05 -0.14
- joint right_camera_joint: origin xyz=0.17 -0.3 1.3 rpy=0 0.05 -3.0 -> xyz=0.1 -0.2 1.15 rpy=0 0.05 -3.0

Commit message: rosbag get param process and param write results to ods done

File: src/prius_description/urdf/prius.urdf (robot description, URDF)
Before this commit: robot solab_prius, 24 links, 23 joints
Joints:
- joint front_camera_joint: origin xyz=0.17 -0.2 1.3 rpy=0 0.05 -1.5707 -> xyz=0.17 -0.2 1.4 rpy=0 0.05 -1.5707
- joint left_camera_joint: origin xyz=0.22 -0.2 1.15 rpy=0 0.05 -0.14 -> xyz=0.17 -0.2 1.4 rpy=0 0.05 -0.0707
- joint right_camera_joint: origin xyz=0.1 -0.2 1.15 rpy=0 0.05 -3.0 -> xyz=0.17 -0.2 1.4 rpy=0 0.05 -3.0707
